Commit message: Calibrated the robot with the inherit motor ability and imu.

File: src/roombabot_description/urdf/roombabot.urdf.xacro (robot description, xacro)
@@ -31,6 +31,6 @@
   <xacro:property name="body_height"     value="0.084"/>
   <xacro:property name="body_mass"       value="3.0"/>
-  <!-- 72 mm diameter drive wheels on a 235 mm track. -->
-  <xacro:property name="wheel_radius"     value="0.036"/>
+  <!-- 64.35 mm diameter drive wheels (caliper, 2026-10-11) on a 235 mm track. -->
+  <xacro:property name="wheel_radius"     value="0.0322"/>
   <xacro:property name="wheel_width"      value="0.025"/>
   <xacro:property name="wheel_separation" value="0.235"/>

File: src/roombabot_description/urdf/roombabot_ros2_control.xacro (robot description, xacro)
@@ -43,6 +43,6 @@
         </xacro:unless>
         <!-- ros2_control Common Interfaces -->
-        <!-- Limits are wheel angular velocity in rad/s. At a 0.036 m wheel radius,
-             15 rad/s is ~0.54 m/s at the rim, comfortably above the 0.4 m/s cap the
+        <!-- Limits are wheel angular velocity in rad/s. At a 0.0322 m wheel radius,
+             15 rad/s is ~0.48 m/s at the rim, comfortably above the 0.4 m/s cap the
              diff_drive_controller applies to the base. -->
         <joint name="wheel_right_joint">

Commit message: Urdf fixes

File: src/roombabot_description/urdf/roombabot.urdf.xacro (robot description, xacro)
@@ -264,9 +264,12 @@
   <!-- Centred on the turning axis: an offset lidar makes the scan appear to swing
        through the map during in-place rotation, which AMCL reads as real motion.
-       The -90 degree yaw matches the RPLIDAR A1's zero-angle mark pointing at the
-       robot's right side when the cable exits to the rear — re-check this against
-       the physical mounting before trusting a map. -->
+       Yaw 180 deg: the lidar's zero angle points to the robot's REAR. Measured
+       2026-10-11 by facing a wall squarely: its normal came out at +174.8 deg in
+       laser_link, and the lidar is visibly square to the chassis, so the ~5 deg is
+       placement error. (The -90 inherited here before was wrong by 90 deg and
+       smeared every map.) Rotation axis confirmed on the turning axis; 0.165 m to
+       the shell edge. -->
   <joint name="laser_joint" type="fixed">
-    <origin xyz="0 0 ${laser_height - base_height}" rpy="0 0 ${-pi/2.0}"/>
+    <origin xyz="0 0 ${laser_height - base_height}" rpy="0 0 ${pi}"/>
     <parent link="base_link"/>
     <child link="laser_link"/>

File: src/roombabot_description/urdf/roombabot_ros2_control.xacro (robot description, xacro)
@@ -25,7 +25,6 @@
                      across boots. -->
                 <param name="port">$(arg motor_port)</param>
-                <!-- Ignored by a native-USB ESP32 (a CDC endpoint has no real baud
-                     rate) but still has to be a value termios accepts, and it
-                     matters if this link ever moves to a hardware UART. -->
+                <!-- Must match Serial.begin() in esp32_motor.ino: the DevKit's CP2102
+                     bridge talks to the ESP32's hardware UART, so the rate is real. -->
                 <param name="baud_rate">921600</param>
                 <!-- Counts per full wheel revolution, after gearing and whatever
